File: prototype/hardware/Kicad/ICSSPicoTracker2/ICSSPicoTracker2.kicad_pcb (KiCad board)
At the start: 2 copper layers, 151 parts, among them J1 Conn_01x04, J2 Conn_01x02, J3 Conn_01x02, Q1 Q_PMOS_DGS, U1 ATSAML21G18B-MUT, U11 74LVC1G04, U12 MAX2659ELT+, U13 SAFEB1G57KE0F00, U14 M8030KT, U15 W25Q16DW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

Commit message: Add Antenna footprints
Parts:
- added ANT2: Johanson868, ICSSPicoTracker2:Johanson868, F.Cu at (-796.3, -535.9)
- added ANT3: Johanson434, ICSSPicoTracker2:Johanson434, F.Cu at (-804.4, -556.3)
- added J4: Conn_01x02, Connector_PinHeader_2.54mm:PinHeader_1x02_P2.54mm_Vertical, F.Cu at (-796.0, -549.1)
- C1, C2, C5, C81, C83, C84, C92: value https://www.murata.com/en-eu/products/productdata/8797690593310/DS-SAFEB1G57KE0F00.pdf?1453347007000 -> 10uF
- moved C92 20.8 mm to (-784.4, -520.7)
- moved C3 18.1 mm to (-774.2, -516.9)
- moved C7 16.2 mm to (-781.5, -530.9)
- moved C6 15.3 mm to (-767.1, -519.2)
- moved U1 14.5 mm to (-773.7, -522.1)
- moved C87 14.4 mm to (-781.6, -525.8)
- moved C5 13.0 mm to (-767.1, -520.7)
- moved C2 12.1 mm to (-781.0, -522.5), turned to 180 degrees
- moved J2 11.8 mm to (-768.4, -523.2), turned to 180 degrees
- moved C9 11.4 mm to (-781.6, -527.0)
- moved C1 10.7 mm to (-774.2, -515.1)
- moved C86 9.45 mm to (-767.1, -515.4)
- moved C93 9.20 mm to (-784.4, -522.5)
- moved R1 8.17 mm to (-781.6, -529.1)
- moved Y3 7.42 mm to (-770.4, -516.1)
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
Commit message: Smaller Antenna and try some layouts
Parts:
- ANT3: value Johanson434 -> Yageo434; footprint ICSSPicoTracker2:Johanson434 -> ICSSPicoTracker2:Yageo434
- X1: footprint Oscillator:Oscillator_SMD_SeikoEpson_SG210-4Pin_2.5x2.0mm -> Oscillator:Oscillator_SMD_IQD_IQXO70-4Pin_7.5x5.0mm
- moved J4 1039.7 mm to (98.0, -18.5), turned to 180 degrees
- moved ANT2 1036.8 mm to (95.8, -7.62), turned to 0 degrees
- moved ANT3 1036.5 mm to (92.5, -36.6)
- moved U5 1017.8 mm to (79.2, -7.62)
- moved C55 1014.8 mm to (89.4, -7.11), turned to 270 degrees
- moved C51 1014.4 mm to (83.6, -7.62), turned to 180 degrees
- moved L17 1012.5 mm to (94.3, -18.5)
- moved C53 1012.3 mm to (85.6, -7.11), turned to 270 degrees
- moved R5 1011.5 mm to (79.0, -11.4)
- moved R3 1010.1 mm to (72.9, -6.60), turned to 180 degrees
- moved C49 1008.7 mm to (80.3, -9.91)
- moved C30 1007.5 mm to (86.9, -19.6), turned to 180 degrees
- moved L19 1007.5 mm to (87.6, -7.62)
- moved C25 1006.6 mm to (85.3, -18.0), turned to 270 degrees
- moved L8 1006.1 mm to (83.8, -18.5)
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Other:
- board outline added: 100 x 40 mm
- copper layers 2 -> 4
- board text added: "Board is 4 layer JLCPCB Type JLC7628 1mm oveall thickness Layer 1 RF and Signal 1oz copper Insulator .2mm 4.6 dielectric constant Layer 2 Ground 1/2 oz copper Insulator 1.065mm 4.6 dielectric constant Layer 3 Power 1/2oz copper Insulator 0.2mm 4.6 dielectric constant Layer 4 Signal 1oz copper Layer 1-2 50 ohm Microstrip width 11.55mil"
- board text added: "Matches should be close to the SX1276 then 50 ohm traces to filters etc."
- board text added: "Maximum board Outline 100mm * 40mm"
